File: Hardware/javi_VCAvolumenContol/javi_VCAvolumenContol_revB.sch (EAGLE design)
At the start: 34 parts, among them J1 EUROPWR_2X05-SMD

Commit message: Bug in the pcb fixed, +12V rail was not connected in both VC in potentiometers. Also i added names to the chip rails
Connections:
- net N$1 renamed SIGNAL_L
- net N$10 renamed BIAS_R
- net N$13 renamed VC_IN_R
- net N$14 renamed VC_IN_L
- net N$2 renamed SIGNAL_R
- net N$22 renamed V-_R
- net N$3 renamed OUT_R
- net N$4 renamed OUT_L
- net N$6 renamed V+_R
- net N$7 renamed V-_L
- net N$8 renamed V+_L
- net N$9 renamed BIAS_L
Changed lines of the file:
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@@
 <?xml version="1.0" encoding="utf-8"?>
 <!DOCTYPE eagle SYSTEM "eagle.dtd">
-<eagle version="9.3.2">
+<eagle version="9.6.2">
 <drawing>
 <settings>
@@
 </segment>
 </net>
-<net name="N$1" class="0">
+<net name="SIGNAL_L" class="0">
 <segment>
 <pinref part="LM13700M" gate="A" pin="IOUT"/>
@@
 <wire x1="114.3" y1="38.1" x2="114.3" y2="40.64" width="0.1524" layer="91"/>
 <junction x="114.3" y="40.64"/>
-</segment>
-</net>
-<net name="N$2" class="0">
+<label x="104.14" y="40.64" size="1.778" layer="95"/>
+</segment>
+</net>
+<net name="SIGNAL_R" class="0">
 <segment>
 <pinref part="LM13700M" gate="B" pin="IOUT"/>
@@
 <wire x1="114.3" y1="-10.16" x2="114.3" y2="-7.62" width="0.1524" layer="91"/>
 <junction x="114.3" y="-7.62"/>
-</segment>
-</net>
-<net name="N$3" class="0">
+<label x="104.14" y="-7.62" size="1.778" layer="95"/>
+</segment>
+</net>
+<net name="OUT_R" class="0">
 <segment>
 <pinref part="LM13700M" gate="BUFB" pin="OUT"/>
@@
 <junction x="144.78" y="-7.62"/>
 <pinref part="COUPLING_C_R" gate="G$1" pin="1"/>
-</segment>
-</net>
-<net name="N$4" class="0">
+<label x="139.7" y="-7.62" size="1.778" layer="95"/>
+</segment>
+</net>
+<net name="OUT_L" class="0">
 <segment>
 <pinref part="LM13700M" gate="BUFA" pin="OUT"/>
@@
 <junction x="144.78" y="40.64"/>
 <pinref part="COUPLING_C_L" gate="G$1" pin="1"/>
+<label x="139.7" y="40.64" size="1.778" layer="95"/>
 </segment>
 </net>
@@
 </segment>
 </net>
-<net name="N$6" class="0">
+<net name="V+_R" class="0">
 <segment>
 <pinref part="RP_R" gate="G$1" pin="2"/>
@@
 <wire x1="35.56" y1="0" x2="43.18" y2="0" width="0.1524" layer="91"/>
 <junction x="43.18" y="0"/>
-</segment>
-</net>
-<net name="N$8" class="0">
+<label x="58.42" y="0" size="1.778" layer="95"/>
+</segment>
+</net>
+<net name="V+_L" class="0">
 <segment>
 <pinref part="RP_L" gate="G$1" pin="2"/>
@@
 <wire x1="35.56" y1="48.26" x2="43.18" y2="48.26" width="0.1524" layer="91"/>
 <junction x="43.18" y="48.26"/>
-</segment>
-</net>
-<net name="N$9" class="0">
+<label x="58.42" y="48.26" size="1.778" layer="95"/>
+</segment>
+</net>
+<net name="BIAS_L" class="0">
 <segment>
 <pinref part="RD_L" gate="G$1" pin="1"/>
 <pinref part="LM13700M" gate="A" pin="BIAS"/>
 <wire x1="60.96" y1="40.64" x2="63.5" y2="40.64" width="0.1524" layer="91"/>
-</segment>
-</net>
-<net name="N$10" class="0">
+<label x="60.96" y="40.64" size="1.778" layer="95"/>
+</segment>
+</net>
+<net name="BIAS_R" class="0">
 <segment>
 <pinref part="RD_R" gate="G$1" pin="1"/>
 <pinref part="LM13700M" gate="B" pin="BIAS"/>
 <wire x1="60.96" y1="-7.62" x2="63.5" y2="-7.62" width="0.1524" layer="91"/>
-</segment>
-</net>
-<net name="N$13" class="0">
+<label x="60.96" y="-7.62" size="1.778" layer="95"/>
+</segment>
+</net>
+<net name="VC_IN_R" class="0">
 <segment>
 <pinref part="RC_R" gate="G$1" pin="1"/>
@@
 <wire x1="33.02" y1="12.7" x2="96.52" y2="12.7" width="0.1524" layer="91"/>
 <wire x1="96.52" y1="12.7" x2="96.52" y2="-2.54" width="0.1524" layer="91"/>
-</segment>
-</net>
-<net name="N$14" class="0">
+<label x="91.44" y="12.7" size="1.778" layer="95"/>
+</segment>
+</net>
+<net name="VC_IN_L" class="0">
 <segment>
 <pinref part="RC_L" gate="G$1" pin="1"/>
@@
 <wire x1="33.02" y1="60.96" x2="96.52" y2="60.96" width="0.1524" layer="91"/>
 <wire x1="96.52" y1="60.96" x2="96.52" y2="45.72" width="0.1524" layer="91"/>
+<label x="91.44" y="60.96" size="1.778" layer="95"/>
 </segment>
 </net>
@@
 </segment>
 </net>
-<net name="N$7" class="0">
+<net name="V-_L" class="0">
 <segment>
 <pinref part="RP_L1" gate="G$1" pin="1"/>
@@
 <pinref part="LM13700M" gate="A" pin="IN-"/>
 <wire x1="60.96" y1="33.02" x2="63.5" y2="33.02" width="0.1524" layer="91"/>
+<label x="58.42" y="33.02" size="1.778" layer="95"/>
 </segment>
 </net>
@@
 </segment>
 </net>
-<net name="N$22" class="0">
+<net name="V-_R" class="0">
 <segment>
 <pinref part="RP_R1" gate="G$1" pin="1"/>
@@
 <pinref part="LM13700M" gate="B" pin="IN-"/>
 <wire x1="55.88" y1="-15.24" x2="63.5" y2="-15.24" width="0.1524" layer="91"/>
-</segment>
-</net>
+<label x="58.42" y="-15.24" size="1.778" layer="95"/>
+</segment>
+</net>
